File: sensorboard.sch (EAGLE design)
At the start: 43 parts, among them U1 LM1117MP-3.3, U2 LM324D

Commit message: routing
Parts:
- removed JP1: (no value), pinhead:PINHD-1X6
- removed JP2: (no value), pinhead:PINHD-1X3
- removed JP3: (no value), pinhead:PINHD-1X16
- removed R19, R2, R20: 10k, rcl:R-EU_R0805
- removed U$4: PCA9532D, philips:PCA9532D
- added U$5: DS18S20, dallas:DS18S20
- U$3: value HOHLBUCHSE -> BMP085; device Ergaenzung:HOHLBUCHSE -> humidity:BMP085
- renumbered JP4 to JP6
Connections:
- removed net !RESET: R20.1, U$4.!RESET
- removed net EOC: JP1.4
- removed net N$10: JP3.3, U$4.LED2
- removed net N$11: JP3.4, U$4.LED3
- removed net N$12: JP3.5, U$4.LED4
- removed net N$13: JP3.6, U$4.LED5
- removed net N$14: JP3.7, U$4.LED6
- removed net N$15: JP3.8, U$4.LED7
- removed net N$16: JP3.9, U$4.LED8
- removed net N$17: JP3.10, U$4.LED9
- removed net N$18: JP3.11, U$4.LED10
- removed net N$19: JP3.12, U$4.LED11
- removed net N$20: JP3.13, U$4.LED12
- removed net N$21: JP3.14, U$4.LED13
- removed net N$22: JP3.15, U$4.LED14
- removed net N$23: JP3.16, U$4.LED15
- removed net N$8: JP3.1, U$4.LED0
- removed net N$9: JP3.2, U$4.LED1
- removed net PF3: U$1.PD3
- removed net XCLR: JP1.3
- net +3V3: now also U$3.VCC, U$5.VDD; no longer JP1.6, JP2.3, R19.2, R2.2, R20.2, U$4.VDD
- net +5V: no longer U$3.I
- net DQ: now also U$5.DQ; no longer JP2.2
- net GND: now also U$3.GND, U$5.GND; no longer JP1.5, JP2.1, U$3.O, U$4.A0, U$4.A1, U$4.A2, U$4.VSS
- net PD3: now also U$1.PD3
- net SCL: now also U$3.SCL; no longer JP1.2, R19.1, U$4.SCL
- net SDA: now also U$3.SDA; no longer JP1.1, R2.1, U$4.SDA
Other:
- note removed: "LED driver"
- moved on the sheet: R12
